Commit message: fix rotation bug

File: URDF_template/preAlphaDrone.urdf (robot description, URDF)
Before this commit: robot quadrotor, 5 links, 4 joints
Joints:
- joint rotor_1_joint: origin xyz=0.1636 0.0485 0.1637 rpy=0 0 0 -> xyz=0.1636 -0.1637 0.0485 rpy=1.5708 0 0
- joint rotor_2_joint: origin xyz=0.1636 0.0485 -0.1637 rpy=0 0 0 -> xyz=0.1636 0.1637 0.0485 rpy=1.5708 0 0
- joint rotor_3_joint: origin xyz=-0.1636 0.0485 -0.1637 rpy=0 0 0 -> xyz=-0.1636 0.1637 0.0485 rpy=1.5708 0 0
- joint rotor_4_joint: origin xyz=-0.1637 0.0485 0.1637 rpy=0 0 0 -> xyz=-0.1637 -0.1637 0.0485 rpy=1.5708 0 0
