Commit message: adapted for the new PX4 LQI+Lyapunov LMI controller

File: simulation/urdf/preBetaDrone.urdf (robot description, URDF)
Before this commit: robot quadrotor, 5 links, 4 joints
Links:
- link base_link: mass 3.0 -> 2.65686; geometry collision mesh filename=../models/Draft10e.stl; visual mesh filename=../models/Draft10e.stl
- link rotor_1: mass 0.05 -> 0.026; geometry collision mesh filename=../models/HQ_0MacroQuad_Prop_10a.stl; visual mesh filename=../models/HQ_0MacroQuad_Prop_10a.stl
- link rotor_2: mass 0.05 -> 0.026; geometry collision mesh filename=../models/HQ_0MacroQuad_Prop_10a.stl; visual mesh filename=../models/HQ_0MacroQuad_Prop_10a.stl
- link rotor_3: mass 0.05 -> 0.026; geometry collision mesh filename=../models/HQ_0MacroQuad_Prop_10a.stl; visual mesh filename=../models/HQ_0MacroQuad_Prop_10a.stl
- link rotor_4: mass 0.05 -> 0.026; geometry collision mesh filename=../models/HQ_0MacroQuad_Prop_10a.stl; visual mesh filename=../models/HQ_0MacroQuad_Prop_10a.stl
Joints:
- joint rotor_1_joint: axis 0 1 0 -> 0 0 1; limit lower=0 upper=10000 effort=1.0 velocity=1000 -> lower=0 upper=1000 effort=1.0 velocity=1000; origin xyz=0.1636 -0.1637 0.0485 rpy=1.5708 0 0 -> xyz=0.1584336 -0.1584337 0.0486 rpy=0 0 0
- joint rotor_2_joint: axis 0 -1 0 -> 0 0 1; limit lower=0 upper=10000 effort=1.0 velocity=1000 -> lower=0 upper=1000 effort=1.0 velocity=1000; origin xyz=0.1636 0.1637 0.0485 rpy=1.5708 0 0 -> xyz=0.1584336 0.1584337 0.0486 rpy=0 0 0
- joint rotor_3_joint: axis 0 1 0 -> 0 0 1; limit lower=0 upper=10000 effort=1.0 velocity=1000 -> lower=0 upper=1000 effort=1.0 velocity=1000; origin xyz=-0.1636 0.1637 0.0485 rpy=1.5708 0 0 -> xyz=-0.1584336 0.1584337 0.0486 rpy=0 0 0
- joint rotor_4_joint: axis 0 -1 0 -> 0 0 1; limit lower=0 upper=10000 effort=1.0 velocity=1000 -> lower=0 upper=1000 effort=1.0 velocity=1000; origin xyz=-0.1637 -0.1637 0.0485 rpy=1.5708 0 0 -> xyz=-0.1584337 -0.1584337 0.0486 rpy=0 0 0
