Commit message: bug fixes

File: simulation/urdf/preAlphaDrone.urdf (robot description, URDF)
Before this commit: robot quadrotor, 5 links, 4 joints
Links:
- link base_link: geometry collision mesh filename=../models/Draft9s.stl; visual mesh filename=../models/Draft9s.stl
- link rotor_1: geometry collision mesh filename=../models/HQ_0MacroQuad_Prop_10.stl; visual mesh filename=../models/HQ_0MacroQuad_Prop_10.stl
- link rotor_2: geometry collision mesh filename=../models/HQ_0MacroQuad_Prop_10.stl; visual mesh filename=../models/HQ_0MacroQuad_Prop_10.stl
- link rotor_3: geometry collision mesh filename=../models/HQ_0MacroQuad_Prop_10.stl; visual mesh filename=../models/HQ_0MacroQuad_Prop_10.stl
- link rotor_4: geometry collision mesh filename=../models/HQ_0MacroQuad_Prop_10.stl; visual mesh filename=../models/HQ_0MacroQuad_Prop_10.stl

Commit message: added stuffs

File: simulation/urdf/preAlphaDrone.urdf (robot description, URDF)
Before this commit: robot quadrotor, 5 links, 4 joints
Joints:
- joint rotor_1_joint: axis 0 0 1 -> 0 1 0; limit lower=0 upper=1000 effort=1.0 velocity=1000 -> lower=0 upper=10000 effort=1.0 velocity=1000
- joint rotor_2_joint: axis 0 0 1 -> 0 -1 0; limit lower=0 upper=1000 effort=1.0 velocity=1000 -> lower=0 upper=10000 effort=1.0 velocity=1000
- joint rotor_3_joint: axis 0 0 1 -> 0 1 0; limit lower=0 upper=1000 effort=1.0 velocity=1000 -> lower=0 upper=10000 effort=1.0 velocity=1000
- joint rotor_4_joint: axis 0 0 1 -> 0 -1 0; limit lower=0 upper=1000 effort=1.0 velocity=1000 -> lower=0 upper=10000 effort=1.0 velocity=1000

Commit message: working

File: simulation/urdf/preAlphaDrone.urdf (robot description, URDF)
Before this commit: robot quadrotor, 5 links, 4 joints
Links:
- link base_link: mass 3.0 -> 0.0
- link rotor_1: mass 0.05 -> 0.0
- link rotor_2: mass 0.05 -> 0.0
- link rotor_3: mass 0.05 -> 0.0
- link rotor_4: mass 0.05 -> 0.0

File: simulation/urdf/preBetaDrone.urdf (robot description, URDF)
Before this commit: robot quadrotor, 5 links, 4 joints
Links:
- link base_link: mass 2.65686 -> 3.18
- link rotor_1: mass 0.026 -> 0.0
- link rotor_2: mass 0.026 -> 0.0
- link rotor_3: mass 0.026 -> 0.0
- link rotor_4: mass 0.026 -> 0.0
